Commit message: fixes for joint traj merging with wam joint state publisher add files from UNIPI repo migrated here

File: soft_hand_description/model/soft_hand.inertia.xacro (robot description, xacro)
@@ -8,7 +8,12 @@
     <!-- conversions -->
     <!-- I couldn't make the simulation work with realistic values, so I tweaked the conversion values -->
+    <!-- use below for the kuka robots -->
     <xacro:property name="mm_to_m" value="0.001"/>
     <xacro:property name="mm2_to_m2" value="0.001"/>
     <xacro:property name="gr_to_Kg" value="0.01"/>
+    <!-- use below for the wam robot -->
+    <!-- <xacro:property name="mm_to_m" value="0.001"/>
+    <xacro:property name="mm2_to_m2" value="0.000001"/>
+    <xacro:property name="gr_to_Kg" value="0.001"/> -->
     <!-- not so negligible, otherwise simulation fails -->
     <xacro:property name="negligible_mass" value="${10*gr_to_Kg}"/>

File: soft_hand_description/model/soft_hand.transmission.xacro (robot description, xacro)
@@ -75,4 +75,16 @@
   <xacro:macro name="soft_hand_transmission" params="name withAdaptiveTransmission">
     <xacro:unless value="${withAdaptiveTransmission}">
+      <!-- work in progress -->
+      <transmission name="${name}_synergy_trans">
+          <robotNamespace>${name}</robotNamespace>
+          <type>transmission_interface/SimpleTransmission</type>
+          <joint name="${name}_synergy_joint">
+            <hardwareInterface>PositionJointInterface</hardwareInterface>
+            <!--hardwareInterface>EffortJointInterface</hardwareInterface-->
+          </joint>
+          <actuator name="${name}_synergy_motor">
+            <mechanicalReduction>1.0</mechanicalReduction>
+          </actuator>
+      </transmission>
       <transmission name="${name}_thumb_abd_trans">
           <robotNamespace>${name}</robotNamespace>

File: soft_hand_description/model/soft_hand.urdf.xacro (robot description, xacro)
@@ -9,5 +9,8 @@
 	<xacro:include filename="$(find soft_hand_description)/model/accesories/kuka_coupler.urdf.xacro"/>
 	<xacro:include filename="$(find soft_hand_description)/model/accesories/clamp.urdf.xacro"/>
+	<xacro:include filename="$(find soft_hand_description)/model/accesories/clamp_30_90.urdf.xacro"/>
 	<xacro:include filename="$(find soft_hand_description)/model/accesories/softhand_base.urdf.xacro"/>
+	<xacro:include filename="$(find soft_hand_description)/model/accesories/merged_angle_flange_30.urdf.xacro"/>
+	<xacro:include filename="$(find soft_hand_description)/model/accesories/merged_angle_flange_90.urdf.xacro"/>
 	<!-- joint properties -->
 	<xacro:property name="abd_lb" value="-30" />
@@ -25,4 +28,5 @@
 	<xacro:property name="damping" value="0.0" />
 	<xacro:property name="friction" value="0.0" />
+	<xacro:property name="pi" value="3.1415926535897931"/>
 	<!-- synergy vector -->
 	<xacro:property name="syn_amp" value="1" />
@@ -394,11 +398,23 @@
 			<xacro:insert_block name="origin"/>
 		</xacro:kuka_coupler>
-		<!-- CLAMP -->
+		<!-- KUKA CLAMP -->
 		<xacro:clamp parent="${name}_kuka_coupler" name="${name}_clamp">
 			<origin xyz="0 0 0.01" rpy="0 0 0"/>
 		</xacro:clamp>
+		<!-- 30 DEG FLANGE -->
+		<xacro:flange_30 parent="${name}_clamp" name="${name}_flange_30">
+			<origin xyz="0 0 0.008" rpy="1.5708 0 1.5708"/>
+		</xacro:flange_30>
+		<!-- CLAMP 30 - 90 -->
+		<xacro:clamp_30_90 parent="${name}_flange_30" name="${name}_clamp_30_90">
+			<origin xyz="0 0.037 0.012" rpy="0 1.0472 1.5708"/>
+		</xacro:clamp_30_90>
+		<!-- 90 DEG FLANGE -->
+		<xacro:flange_90 parent="${name}_clamp_30_90" name="${name}_flange_90">
+			<origin xyz="0.06 0.00 0.008" rpy="1.5708 0 -1.5708"/>
+		</xacro:flange_90>
 		<!-- SOFT HAND BASE -->
-		<xacro:softhand_base parent="${name}_clamp" name="${name}_softhand_base" left="${left}">
-			<origin xyz="0 0 0.004" rpy="0 0 0"/>
+		<xacro:softhand_base parent="${name}_flange_90" name="${name}_softhand_base" left="${left}">
+			<origin xyz="0 0.03 0.120" rpy="0 3.1415 -1.5708"/>
 		</xacro:softhand_base>
 		<!-- PALM -->
